File: Led Heart.kicad_pcb (KiCad board)
At the start: 2 copper layers, 41 parts, among them J1 Conn_01x01_Female, J2 Conn_01x01_Female, J3 Conn_01x01_Female, SW1 SW_DIP_x01, U1 STM32L031G6U6

Commit message: poprawki
Parts:
- added G***: LOGO, LOGO, F.Cu at (107.0, 96.0)
- D1, D10, D11, D12, D13, D14, D15, D16, D17, D18, D2, D3, D4, D5, D6, D7, D8, D9: footprint LED_SMD:LED_0603_1608Metric -> Diode_SMD:D_0805_2012Metric
- R1, R10, R11, R12, R13, R14, R15, R16, R17, R18, R2, R3, R4, R5, R6, R7, R8, R9: footprint LED_SMD:LED_0603_1608Metric -> Resistor_SMD:R_0805_2012Metric
- moved D1 11.8 mm to (94.0, 92.2)
- moved R1 11.8 mm to (97.9, 92.4)
- moved D2 9.67 mm to (94.4, 88.8)
- moved R2 9.67 mm to (98.5, 88.5)
- moved SW1 3.97 mm to (106.8, 103.2)
- moved U1 3.97 mm to (106.8, 96.1)
- moved J3 3.97 mm to (109.9, 92.3)
- moved J1 3.97 mm to (111.1, 94.1)
- moved J2 3.97 mm to (111.6, 98.7)
Other:
- board outline added: 30.5 x 27.2 mm

Commit message: kk
Parts:
- removed J3: Conn_01x01_Female, Connector_PinHeader_1.00mm:PinHeader_1x01_P1.00mm_Vertical
- added C1: 100nF, Capacitor_SMD:C_1206_3216Metric, F.Cu at (112.0, 91.9)
- added C2: 100nF, Capacitor_SMD:C_1206_3216Metric, F.Cu at (106.4, 91.9)
- added C3: 100nF, Capacitor_SMD:C_1206_3216Metric, F.Cu at (100.7, 95.3)
- added R19: 100k, Capacitor_SMD:C_1206_3216Metric, F.Cu at (100.7, 91.9)
- added R20: 100k, Capacitor_SMD:C_1206_3216Metric, F.Cu at (106.4, 95.3)
- added R21: 100k, Capacitor_SMD:C_1206_3216Metric, F.Cu at (112.0, 95.3)
- R1, R10, R11, R12, R13, R14, R15, R16, R17, R18, R2, R3, R4, R5, R6, R7, R8, R9: value R -> 3.3k; footprint Resistor_SMD:R_0805_2012Metric -> Resistor_SMD:R_0402_1005Metric
- SW1: footprint Connector_PinHeader_1.00mm:PinHeader_2x02_P1.00mm_Vertical_SMD -> Button_Switch_SMD:SW_SPST_TL3342
- moved D5 15.8 mm to (106.9, 87.1)
- moved R5 15.2 mm to (106.9, 88.9), turned to 180 degrees
- moved D6 13.5 mm to (114.0, 83.6), turned to 180 degrees
- moved R4 12.1 mm to (102.9, 84.1)
- moved R6 10.0 mm to (110.7, 85.3), turned to 180 degrees
- moved D3 9.66 mm to (96.3, 85.9)
- moved R3 8.18 mm to (99.1, 85.3)
- moved D4 6.71 mm to (100.1, 83.8), turned to 180 degrees
- moved R1 4.52 mm to (94.0, 90.2)
- moved R2 1.49 mm to (97.3, 87.6)
- moved D2 0.64 mm to (94.5, 88.1)
- moved SW1 0.55 mm to (107.2, 103.6), turned to 0 degrees
- turned D1 to 180 degrees
Connections:
- D1 pad 1: unconnected-(D1-Pad1) -> Net-(U1-Pad6)
- U1 pad 21: Net-(J1-Pad1) -> Net-(U1-Pad21)
- U1 pad 6: unconnected-(U1-Pad6) -> Net-(U1-Pad6)

Commit message: Uporządkowanie pcb diody w trakcie podłączania
Parts:
- C1, C2, C3: footprint Capacitor_SMD:C_1206_3216Metric -> Capacitor_SMD:C_0402_1005Metric
- J1: value Conn_01x01_Female -> Conn_01x03_Female; footprint Connector_PinHeader_1.00mm:PinHeader_1x01_P1.00mm_Vertical -> Connector_PinHeader_1.00mm:PinHeader_1x03_P1.00mm_Vertical_SMD_Pin1Left; moved to B.Cu
- J2: value Conn_01x01_Female -> Conn_01x02_Female; footprint Connector_PinHeader_1.00mm:PinHeader_1x01_P1.00mm_Vertical -> Battery:BatteryHolder_MPD_BC2003_1x2032; moved to B.Cu
- R19, R20, R21: value 100k -> 10k; footprint Capacitor_SMD:C_1206_3216Metric -> Resistor_SMD:R_0402_1005Metric
- moved D15 38.6 mm to (71.2, 104.9)
- moved R15 38.6 mm to (71.6, 101.9)
- moved R14 21.0 mm to (98.0, 100.8)
- moved D14 20.0 mm to (97.8, 99.3), turned to 180 degrees
- moved D16 17.9 mm to (85.6, 117.3)
- moved D17 17.9 mm to (81.1, 114.1)
- moved R17 17.9 mm to (80.0, 116.7)
- moved R16 17.9 mm to (86.2, 121.7)
- moved D9 17.6 mm to (119.1, 94.7)
- moved R13 17.4 mm to (101.3, 104.4), turned to 180 degrees
- moved D13 17.3 mm to (101.1, 102.9)
- moved R12 16.8 mm to (106.9, 108.5), turned to 180 degrees
- moved R10 16.7 mm to (116.6, 100.6)
- moved R7 16.6 mm to (119.4, 87.9)
- moved R9 15.9 mm to (119.4, 96.3), turned to 180 degrees
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Connections:
- C3 pad 2: Net-(C3-Pad2) -> Net-(U1-Pad10)
- D14 pad 1: unconnected-(D14-Pad1) -> Net-(U1-Pad7)
- J2 pad 1: GND -> +3V0
- R20 pad 1: Net-(C3-Pad2) -> Net-(U1-Pad10)
- SW1 pad 2: Net-(C3-Pad2) -> Net-(U1-Pad10)
- U1 pad 10: unconnected-(U1-Pad10) -> Net-(U1-Pad10)
- U1 pad 21: Net-(U1-Pad21) -> Net-(J1-Pad1)
- U1 pad 22: Net-(U1-Pad22) -> Net-(J1-Pad3)
- U1 pad 7: unconnected-(U1-Pad7) -> Net-(U1-Pad7)
Routing:
- net +3V0: track 0.00 -> 144.7 mm, vias 0 -> 12
- net GND: track 0.00 -> 49.1 mm, vias 0 -> 5
- net (no net): track 0.00 -> 16.4 mm, vias 0 -> 2
- net Net-(U1-Pad7): track 0.00 -> 14.6 mm
- net unconnected-(D13-Pad1): track 0.00 -> 11.4 mm
- net unconnected-(D4-Pad1): track 0.00 -> 9.98 mm
- net unconnected-(D3-Pad1): track 0.00 -> 9.58 mm
- net Net-(D1-Pad1): track 0.00 -> 9.48 mm
- net Net-(J1-Pad1): track 0.00 -> 8.11 mm, vias 0 -> 1
- net Net-(C2-Pad1): track 0.00 -> 7.59 mm
- net Net-(U1-Pad10): track 0.00 -> 6.60 mm
- net unconnected-(D5-Pad1): track 0.00 -> 5.06 mm
- net Net-(D5-Pad2): track 0.00 -> 2.12 mm
- net Net-(D4-Pad2): track 0.00 -> 1.96 mm
- net Net-(D8-Pad2): track 0.00 -> 1.91 mm
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Other:
- outline, holes or cut-outs redrawn

Commit message: k
Parts:
- removed D15, D16, D17, D18: LED, Diode_SMD:D_0805_2012Metric
- removed G***: LOGO, LOGO
- removed R15, R16, R17, R18: 3.3k, Resistor_SMD:R_0402_1005Metric
- J2: footprint Battery:BatteryHolder_MPD_BC2003_1x2032 -> SamacSys_Parts:BatteryHolder_MPD_BC2003_1x2032
- moved J1 0.26 mm to (112.0, 85.3)
Connections:
- D10 pad 1: unconnected-(D10-Pad1) -> Net-(U1-Pad14)
- D11 pad 1: unconnected-(D11-Pad1) -> Net-(U1-Pad13)
- D12 pad 1: unconnected-(D12-Pad1) -> Net-(U1-Pad12)
- D13 pad 1: unconnected-(D13-Pad1) -> Net-(D13-Pad1)
- D2 pad 1: unconnected-(D2-Pad1) -> Net-(U1-Pad8)
- D3 pad 1: unconnected-(D3-Pad1) -> Net-(D3-Pad1)
- D4 pad 1: unconnected-(D4-Pad1) -> Net-(D4-Pad1)
- D5 pad 1: unconnected-(D5-Pad1) -> Net-(U1-Pad23)
- D6 pad 1: unconnected-(D6-Pad1) -> Net-(U1-Pad20)
- D7 pad 1: unconnected-(D7-Pad1) -> Net-(U1-Pad19)
- D8 pad 1: unconnected-(D8-Pad1) -> Net-(U1-Pad18)
- D9 pad 1: unconnected-(D9-Pad1) -> Net-(U1-Pad15)
- U1 pad 12: unconnected-(U1-Pad12) -> Net-(U1-Pad12)
- U1 pad 13: unconnected-(U1-Pad13) -> Net-(U1-Pad13)
- U1 pad 14: unconnected-(U1-Pad14) -> Net-(U1-Pad14)
- U1 pad 15: unconnected-(U1-Pad15) -> Net-(U1-Pad15)
- U1 pad 18: unconnected-(U1-Pad18) -> Net-(U1-Pad18)
- U1 pad 19: unconnected-(U1-Pad19) -> Net-(U1-Pad19)
- U1 pad 2: unconnected-(U1-Pad2) -> Net-(D4-Pad1)
- U1 pad 20: unconnected-(U1-Pad20) -> Net-(U1-Pad20)
- U1 pad 23: unconnected-(U1-Pad23) -> Net-(U1-Pad23)
- U1 pad 3: unconnected-(U1-Pad3) -> Net-(D3-Pad1)
- U1 pad 8: unconnected-(U1-Pad8) -> Net-(U1-Pad8)
- U1 pad 9: unconnected-(U1-Pad9) -> Net-(D13-Pad1)
Routing:
- net Net-(U1-Pad8): track 0.00 -> 18.7 mm, vias 0 -> 2
- net (no net): track 16.4 -> 0.00 mm, vias 2 -> 0
- net GND: track 49.1 -> 65.5 mm, vias 5 -> 6
- net Net-(U1-Pad12): track 0.00 -> 12.9 mm
- net Net-(D13-Pad1): track 0.00 -> 12.8 mm
- net Net-(U1-Pad13): track 0.00 -> 11.6 mm
- net unconnected-(D13-Pad1): track 11.4 -> 0.00 mm
- net Net-(U1-Pad19): track 0.00 -> 11.2 mm
- net Net-(U1-Pad18): track 0.00 -> 11.2 mm
- net Net-(U1-Pad20): track 0.00 -> 11.1 mm
- net Net-(D4-Pad1): track 0.00 -> 10.8 mm
- net Net-(D3-Pad1): track 0.00 -> 10.7 mm
- net unconnected-(D4-Pad1): track 9.98 -> 0.00 mm
- net unconnected-(D3-Pad1): track 9.58 -> 0.00 mm
- net Net-(U1-Pad15): track 0.00 -> 9.40 mm
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Other:
- board size 30.5 x 27.2 mm -> 32.2 x 28.7 mm

Commit message: dodałem przypadkiem tez emila projekt ale moj ma tez duzo aktualizacji tutaj
Parts:
- J2: footprint SamacSys_Parts:BatteryHolder_MPD_BC2003_1x2032 -> Battery:BatteryHolder_MPD_BC2003_1x2032
- moved D5 0.16 mm to (106.9, 86.7)
Routing:
- net +3V0: track 145.0 -> 143.3 mm
Other:
- outline, holes or cut-outs redrawn

Commit message: Usuniety projekt emila dodany przypadkiem i ostatnie chyba poprawki
Parts:
- added REF**: MountingHole_2.1mm, MountingHole:MountingHole_2.1mm, F.Cu at (106.9, 84.4)
- J2: footprint Battery:BatteryHolder_MPD_BC2003_1x2032 -> SamacSys_Parts:BatteryHolder_MPD_BC2003_1x2032
- moved J1 3.33 mm to (115.3, 85.2)
- moved J2 0.39 mm to (107.1, 94.9)
- moved D6 0.24 mm to (114.0, 83.8)
Routing:
- net Net-(J1-Pad3): track 7.43 -> 10.7 mm
- net +3V0: track 143.3 -> 146.5 mm, vias 12 -> 13
- net GND: track 65.5 -> 67.4 mm
Other:
- outline, holes or cut-outs redrawn

Commit message: okkk
Parts:
- moved R1 0.26 mm to (94.7, 96.3)
Changed lines of the file:
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@@
   )
   (footprint "Resistor_SMD:R_0402_1005Metric" (layer "F.Cu")
-    (at 94.742 96.52)
+    (at 94.742 96.26)
     (descr "Resistor SMD 0402 (1005 Metric), square (rectangular) end terminal, IPC_7351 nominal, (Body size source: IPC-SM-782 page 72, https://www.pcb-3d.com/wordpress/wp-content/uploads/ipc-sm-782a_amendment_1_and_2.pdf), generated with kicad-footprint-generator")
     (tags "resistor")
@@
   (gr_line (start 98.953544 80.800999) (end 99.161225 80.786298) (layer "Edge.Cuts") (width 0.1))
   (segment (start 94.232 94.9155) (end 94.0585 94.742) (width 0.25) (layer "F.Cu") (net 1))
-  (segment (start 94.232 96.52) (end 94.232 94.9155) (width 0.25) (layer "F.Cu") (net 1))
+  (segment (start 94.232 96.26) (end 94.232 94.9155) (width 0.25) (layer "F.Cu") (net 1))
   (segment (start 93.728 89.7385) (end 92.7885 90.678) (width 0.25) (layer "F.Cu") (net 2))
   (segment (start 93.728 89.154) (end 93.728 89.7385) (width 0.25) (layer "F.Cu") (net 2))
@@
   (segment (start 104.562 106.968479) (end 106.051521 108.458) (width 0.2) (layer "F.Cu") (net 16))
   (segment (start 109.728 84.074) (end 109.22 84.582) (width 0.25) (layer "F.Cu") (net 16))
+  (segment (start 95.252 97.212) (end 95.252 96.26) (width 0.25) (layer "F.Cu") (net 16))
   (segment (start 103.634 84.074) (end 104.14 84.074) (width 0.25) (layer "F.Cu") (net 16))
   (segment (start 96.99 93) (end 97.026 92.964) (width 0.25) (layer "F.Cu") (net 16))
@@
   (segment (start 97.5 93.9) (end 97.026 93.426) (width 0.25) (layer "F.Cu") (net 16))
   (segment (start 110.488 84.074) (end 109.728 84.074) (width 0.25) (layer "F.Cu") (net 16))
-  (segment (start 95.252 97.448) (end 95.2 97.5) (width 0.25) (layer "F.Cu") (net 16))
   (segment (start 104.9909 93.209999) (end 104.282102 93.209999) (width 0.25) (layer "F.Cu") (net 16))
   (segment (start 104.648 86.888) (end 104.648 90.9941) (width 0.2) (layer "F.Cu") (net 16))
@@
   (segment (start 118.872 97.282) (end 118.872 96.268) (width 0.2) (layer "F.Cu") (net 16))
   (segment (start 104.648 86.888) (end 104.648 87.023834) (width 0.25) (layer "F.Cu") (net 16))
-  (segment (start 95.252 96.52) (end 95.252 97.448) (width 0.25) (layer "F.Cu") (net 16))
   (segment (start 98.1 101.9) (end 98.1 101.292) (width 0.25) (layer "F.Cu") (net 16))
   (segment (start 92.716 87.884) (end 92.5 88.1) (width 0.25) (layer "F.Cu") (net 16))
@@
   (via (at 118.11 92.964) (size 0.8) (drill 0.4) (layers "F.Cu" "B.Cu") (net 16))
   (via (at 104.648 84.582) (size 0.8) (drill 0.4) (layers "F.Cu" "B.Cu") (net 16))
-  (via (at 95.2 97.5) (size 0.8) (drill 0.4) (layers "F.Cu" "B.Cu") (net 16))
+  (via (at 95.252 97.212) (size 0.8) (drill 0.4) (layers "F.Cu" "B.Cu") (net 16))
   (via (at 118.872 97.282) (size 0.8) (drill 0.4) (layers "F.Cu" "B.Cu") (net 16))
   (segment (start 104.648 84.582) (end 106.225001 83.004999) (width 0.25) (layer "B.Cu") (net 16))

Commit message: kk
Other:
- board text added: "JLCJLCJLCJLC"
Changed lines of the file:
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@@
   (gr_line (start 93.988288 82.890053) (end 94.374347 82.583408) (layer "Edge.Cuts") (width 0.1))
   (gr_line (start 98.953544 80.800999) (end 99.161225 80.786298) (layer "Edge.Cuts") (width 0.1))
+  (gr_text "JLCJLCJLCJLC" (at 98.59 85.02) (layer "B.SilkS")
+    (effects (font (size 1 1) (thickness 0.15)) (justify mirror))
+  )
   (segment (start 94.232 94.9155) (end 94.0585 94.742) (width 0.25) (layer "F.Cu") (net 1))
   (segment (start 94.232 96.26) (end 94.232 94.9155) (width 0.25) (layer "F.Cu") (net 1))
